Commit message: yam

File: models/YAM_umi.urdf (robot description, URDF)
Before this commit: robot YAM_umi, 8 links, 7 joints
Links:
- link base_link: mass 0.46369 -> 0.47109
- link link2: mass 1.0796 -> 1.0928
- link link3: mass 0.5829 -> 0.596
- link link4: mass 0.3896 -> 0.4041
- link link5: mass 0.3686 -> 0.3759
